Commit message: Add files via upload

File: hector_quadrotor/hector_quadrotor_description/urdf/quadrotor_base.urdf.xacro (robot description, xacro)
@@ -24,4 +24,27 @@
       </collision>
     </link>
+    <link name="fixedarm_link">
+        <visual>
+          <origin rpy="0 0 0" xyz="0 0 -0.03" />
+          <geometry>
+            <cylinder radius="0.01" length="0.06"/>
+          </geometry>
+        </visual>
+        <collision>
+          <origin rpy="0 0 0" xyz="0 0 -0.03" />
+          <geometry>
+            <cylinder radius="0.01" length="0.06"/>
+          </geometry>
+        </collision>
+        <inertial>
+          <mass value="0.001"/>
+          <inertia ixx="0.000000325" ixy="0.0" ixz="0.0" iyy="0.000000325" iyz="0.0" izz="0.00000005"/>
+        </inertial>
+      </link>
+      <joint name="fixedarm_joint" type="fixed">
+        <parent link="base_link" />
+        <child link="fixedarm_link"/>
+        <origin xyz="0 0 -0.03" />
+      </joint>
     <!-- Sonar height sensor -->
     <xacro:sonar_sensor name="sonar" parent="base_link" ros_topic="sonar_height" update_rate="10" min_range="0.03" max_range="3.0" field_of_view="${40*pi/180}" ray_count="3">

File: hector_quadrotor/hector_quadrotor_description/urdf/quadrotor_with_asus_with_hokuyo_utm30lx.urdf.xacro (robot description, xacro)
@@ -14,5 +14,5 @@
     <xacro:include filename="$(find hector_sensors_description)/urdf/asus_camera.urdf.xacro" />
     <xacro:asus_camera name="camera" parent="base_link">
-      <origin xyz="0.1 0.0 -0.03" rpy="0 ${M_PI/9} 0"/>
+      <origin xyz="0.1 0.0 -0.04" rpy="0 0 0"/>
     </xacro:asus_camera>
 </robot>

File: hector_quadrotor/hector_quadrotor_description/urdf/quadrotor_with_kinect.urdf.xacro (robot description, xacro)
@@ -8,6 +8,49 @@
     <!-- Kinect -->
     <xacro:include filename="$(find hector_sensors_description)/urdf/kinect_camera.urdf.xacro" />
-    <xacro:kinect_camera name="camera" parent="base_link">
-      <origin xyz="0.23 0.0 -0.1" rpy="0 0 0"/>
+    <link name="movable_link">
+        <visual>
+            <origin rpy="1.5707963267948966 0 0" xyz="0 0 0" />
+            <geometry>
+                <cylinder length="0.01" radius="0.03" />
+            </geometry>
+        </visual>
+        <collision>
+            <origin rpy="1.5707963267948966 0 0" xyz="0 0 0" />
+            <geometry>
+                <cylinder length="0.01" radius="0.03" />
+            </geometry>
+        </collision>
+        <inertial>
+            <mass value="0.1" />
+            <inertia ixx="0.03" iyy="0.03" izz="0.03" ixy="0.0" ixz="0.0" iyz="0.0" />
+        </inertial>
+    </link>
+    <joint name="movable_camera_joint" type="revolute">
+        <origin rpy="0.0 0.0 0.0" xyz="0 0 -0.055" />
+        <parent link="fixedarm_link" />
+        <child link="movable_link" />
+        <axis xyz="0 -1 0" />
+        <limit effort="2" lower="-1.5707963267948966" upper="0" velocity="2.0" />
+    </joint>
+    <xacro:kinect_camera name="camera" parent="movable_link">
+      <origin xyz="0.06 0.0 -0.03" rpy="0 0 0"/>
     </xacro:kinect_camera>
+    <transmission name="trans_movable_camera_joint">
+        <type>transmission_interface/SimpleTransmission</type>
+        <joint name="movable_camera_joint">
+            <hardwareInterface>hardware_interface/PositionJointInterface</hardwareInterface>
+        </joint>
+        <actuator name="movable_camera_joint_motor">
+            <hardwareInterface>hardware_interface/PositionJointInterface</hardwareInterface>
+            <mechanicalReduction>1</mechanicalReduction>
+        </actuator>
+    </transmission>
+    <!--<xacro:kinect_camera name="camera" parent="base_link">
+        <origin xyz="0.23 0.0 -0.1" rpy="0 0 0"/>
+    </xacro:kinect_camera>-->
+    <!--<gazebo>
+        <plugin name="gazebo_ros_control" filename="libgazebo_ros_control.so">
+            <robotNamespace>/</robotNamespace>
+        </plugin>
+    </gazebo>-->
 </robot>
